File: mammut/mammut.kicad_sch (KiCad schematic)
At the start: 31 parts

Commit message: prepare for plotting
Parts:
- C1, C3, C8, C9: value (none) -> 100uF; footprint (none) -> Capacitor_SMD:CP_Elec_6.3x7.7
- C10, C2: value (none) -> 10nF; footprint (none) -> Capacitor_SMD:C_0805_2012Metric
- C4: value (none) -> 33nF; footprint (none) -> Capacitor_SMD:C_0805_2012Metric
- C5, C7: value (none) -> 220nF; footprint (none) -> Capacitor_SMD:C_0805_2012Metric
- C6: value (none) -> 68nF; footprint (none) -> Capacitor_SMD:C_0805_2012Metric
- D1: value (none) -> 1N4007; footprint (none) -> Diode_THT:D_DO-41_SOD81_P10.16mm_Horizontal
- FUZZ1: value (none) -> C5K; footprint (none) -> Potentiometer_THT:Potentiometer_Alpha_RD901F-40-00D_Single_Vertical_CircularHoles
- IN1: value (none) -> IN; footprint (none) -> Connector_Audio:Jack_6.35mm_Neutrik_NMJ4HCD2_Horizontal
- J1: value (none) -> TO FOOTSWITCH; footprint (none) -> Connectors:1X06
- OUT1: value (none) -> OUT; footprint (none) -> Connector_Audio:Jack_6.35mm_Neutrik_NMJ4HCD2_Horizontal
- POWER1: value (none) -> POWER; footprint (none) -> Connector_JST:JST_EH_B2B-EH-A_1x02_P2.50mm_Vertical
- PW1: value (none) -> B500K; footprint (none) -> Potentiometer_THT:Potentiometer_Alpha_RD901F-40-00D_Single_Vertical_CircularHoles
- Q1, Q2: value (none) -> TRANS_NPN-P2N2222A; footprint (none) -> Package_TO_SOT_THT:TO-92L_Inline
- R1, R6: value (none) -> 100; footprint (none) -> Resistor_SMD:R_0805_2012Metric
- R2: value (none) -> 22K; footprint (none) -> Resistor_SMD:R_0805_2012Metric
- R3: value (none) -> 10K; footprint (none) -> Resistor_SMD:R_0805_2012Metric
- R4: value (none) -> 56K; footprint (none) -> Resistor_SMD:R_0805_2012Metric
- R5: value (none) -> 5.1K; footprint (none) -> Resistor_SMD:R_0805_2012Metric
- R7: value (none) -> 100K; footprint (none) -> Resistor_SMD:R_0805_2012Metric
- R8: value (none) -> 2.2K; footprint (none) -> Resistor_SMD:R_0805_2012Metric
- REL/PSH1: value (none) -> B100K; footprint (none) -> Potentiometer_THT:Potentiometer_Alpha_RD901F-40-00D_Single_Vertical_CircularHoles
- SW1: value (none) -> SPDT; footprint (none) -> Connectors:1X03
- TONE1, VOL1: value (none) -> B10K; footprint (none) -> Potentiometer_THT:Potentiometer_Alpha_RD901F-40-00D_Single_Vertical_CircularHoles
Other:
- title: (none) -> Mammut
